Commit message: bad thruster values

File: urdf/robots/lanturn_description/urdf/lanturn.xacro (robot description, xacro)
@@ -124,31 +124,35 @@
     </xacro:thruster_module_first_order_basic_fcn_macro>
   </xacro:macro>
-  <!-- Port-Aft -->
+  <!-- Thruster 0 - Vertical Front Right -->
   <xacro:thruster_macro thruster_id="0">
-    <origin xyz="-1.2 0.415 0.09" rpy="${0*d2r} ${0*d2r} ${-150.0*d2r}"/>
+    <origin xyz="-0.3872 0.06294 0.22092" rpy="${0*d2r} ${0*d2r} ${-30.0*d2r}"/>
   </xacro:thruster_macro>
-  <!-- Starboard-Aft -->
+  <!-- Thruster 1 - Horizontal Front Right-->
   <xacro:thruster_macro thruster_id="1">
-    <origin xyz="-1.2 -0.41 0.09" rpy="${0*d2r} ${0*d2r} ${150.0*d2r}"/>
+    <origin xyz="-0.29064 0.06710 0.15054" rpy="${0*d2r} ${0*d2r} ${-150.0*d2r}"/>
   </xacro:thruster_macro>
-  <!-- Port-Forward -->
+  <!-- Thruster 2 - Vertical Back Right -->
   <xacro:thruster_macro thruster_id="2">
-    <origin xyz="0.95 0.56 -0.61" rpy="${0*d2r} ${0*d2r} ${-30.0*d2r}"/>
+    <origin xyz="-0.38659 0.06199 -0.23044" rpy="${0*d2r} ${0*d2r} ${30.0*d2r}"/>
   </xacro:thruster_macro>
-  <!-- Starboard-Forward -->
+  <!-- Thruster 3 - Horizontal Back Right-->
   <xacro:thruster_macro thruster_id="3">
-    <origin xyz="0.95 -0.56 -0.61" rpy="${0*d2r} ${0*d2r} ${30.0*d2r}"/>
+    <origin xyz="-0.28470 0.06560 -0.016626" rpy="${0*d2r} ${0*d2r} ${150.0*d2r}"/>
   </xacro:thruster_macro>
-  <!-- Port-Forward-Vertical -->
+  <!-- Thruster 4 - Vertical Back Left -->
   <xacro:thruster_macro thruster_id="4">
-    <origin xyz="1.0 0.4 0.5" rpy="${0*d2r} ${90.0*d2r} ${0*d2r}"/>
+    <origin xyz="0.3965 0.06271 -0.23105" rpy="${0*d2r} ${90.0*d2r} ${0*d2r}"/>
   </xacro:thruster_macro>
-  <!-- Starboard-Forward-Vertical -->
+  <!-- Thruster 5 - Horizontal Back Left -->
   <xacro:thruster_macro thruster_id="5">
-    <origin xyz="1.0 -0.4 0.5" rpy="${0*d2r} ${90.0*d2r} ${0*d2r}"/>
+    <origin xyz="0.29505 0.06907 -0.16581" rpy="${0*d2r} ${90.0*d2r} ${0*d2r}"/>
   </xacro:thruster_macro>
-  <!-- Aft-Vertical -->
+  <!-- Thruster 6 - Vertical Front Left -->
   <xacro:thruster_macro thruster_id="6">
-    <origin xyz="-1.25 0.0 0.65" rpy="${0*d2r} ${90.0*d2r} ${0*d2r}"/>
+    <origin xyz="0.39685 0.06564 0.22015" rpy="${0*d2r} ${90.0*d2r} ${0*d2r}"/>
+  </xacro:thruster_macro>
+  <!-- Thruster 7 - Horizontal Front Left -->
+  <xacro:thruster_macro thruster_id="7">
+    <origin xyz="0.30146 0.06198 0.14961" rpy="${0*d2r} ${90.0*d2r} ${0*d2r}"/>
   </xacro:thruster_macro>
  <!-- Default joint state publisher -->

Commit message: new lanturn model, fix robot height over estimation, add thruter png

File: urdf/robots/lanturn_description/urdf/lanturn.xacro (robot description, xacro)
@@ -29,5 +29,5 @@
     </inertial>
     <visual>
-      <origin xyz="0 0 -0.9" rpy="0 0 1.5708"/>
+      <origin xyz="0 0 0" rpy="0 0 1.5708"/>
       <geometry>
         <mesh filename="package://lanturn_description/meshes/lanturn.dae" scale="1 1 1"/>
@@ -35,5 +35,5 @@
     </visual>
     <collision>
-      <origin xyz="0 0 -0.9" rpy="0 0 1.5708"/>
+      <origin xyz="0 0 0" rpy="0 0 1.5708"/>
       <geometry>
         <mesh filename="package://lanturn_description/meshes/lanturn.dae" scale="1 1 1"/>
@@ -103,5 +103,5 @@
  <xacro:include filename="$(find uuv_gazebo_ros_plugins)/urdf/thruster_snippets.xacro"/>
  <!-- Substitute the ECA A9 prop mesh for the larger uuv_descriptions one -->
- <xacro:property name="prop_mesh_file" value="file://$(find eca_a9_description)/mesh/eca_a9_propeller.dae"/>
+ <xacro:property name="prop_mesh_file" value="file://$(find lanturn_description)/meshes/t200_prop.dae"/>
   <!-- Thruster joint and link snippet
        Wrapper for the the thruster_module_first_order_basic_fcn_macro
@@ -130,17 +130,17 @@
   <!-- Thruster 0 - Vertical Starboard-Forward -->
   <xacro:thruster_macro thruster_id="0">
-    <origin xyz="0.385 0.22 -0.859" rpy="${0*d2r} ${-90*d2r} ${0*d2r}"/>
+    <origin xyz="0.385 0.22 0.041" rpy="${0*d2r} ${-90*d2r} ${0*d2r}"/>
   </xacro:thruster_macro>
   <!-- Thruster 1 - Vertical Starboard-Aft -->
   <xacro:thruster_macro thruster_id="1">
-    <origin xyz="0.385 -0.22 -0.859" rpy="${0*d2r} ${-90*d2r} ${0*d2r}"/>
+    <origin xyz="0.385 -0.22 0.041" rpy="${0*d2r} ${-90*d2r} ${0*d2r}"/>
   </xacro:thruster_macro>
   <!-- Thruster 2 - Vertical Port-Forward -->
   <xacro:thruster_macro thruster_id="2">
-    <origin xyz="-0.385 0.22 -0.859" rpy="${0*d2r} ${-90*d2r} ${0*d2r}"/>
+    <origin xyz="-0.385 0.22 0.041" rpy="${0*d2r} ${-90*d2r} ${0*d2r}"/>
   </xacro:thruster_macro>
   <!-- Thruster 3 - Vertical Port-Aft -->
   <xacro:thruster_macro thruster_id="3">
-    <origin xyz="-0.385 -0.22 -0.859" rpy="${0*d2r} ${-90*d2r} ${0*d2r}"/>
+    <origin xyz="-0.385 -0.22 0.041" rpy="${0*d2r} ${-90*d2r} ${0*d2r}"/>
   </xacro:thruster_macro>
  <!-- Default joint state publisher -->

File: urdf/robots/wailord_description/urdf/wailord.xacro (robot description, xacro)
@@ -123,36 +123,4 @@
     </xacro:thruster_module_first_order_basic_fcn_macro>
   </xacro:macro>
-  <!-- Thruster 0 - Vertical Front Right -->
-  <xacro:thruster_macro thruster_id="0">
-    <origin xyz="-0.3872 0.06294 0.22092" rpy="${0*d2r} ${0*d2r} ${-30.0*d2r}"/>
-  </xacro:thruster_macro>
-  <!-- Thruster 1 - Horizontal Front Right-->
-  <xacro:thruster_macro thruster_id="1">
-    <origin xyz="-0.29064 0.06710 0.15054" rpy="${0*d2r} ${0*d2r} ${-150.0*d2r}"/>
-  </xacro:thruster_macro>
-  <!-- Thruster 2 - Vertical Back Right -->
-  <xacro:thruster_macro thruster_id="2">
-    <origin xyz="-0.38659 0.06199 -0.23044" rpy="${0*d2r} ${0*d2r} ${30.0*d2r}"/>
-  </xacro:thruster_macro>
-  <!-- Thruster 3 - Horizontal Back Right-->
-  <xacro:thruster_macro thruster_id="3">
-    <origin xyz="-0.28470 0.06560 -0.016626" rpy="${0*d2r} ${0*d2r} ${150.0*d2r}"/>
-  </xacro:thruster_macro>
-  <!-- Thruster 4 - Vertical Back Left -->
-  <xacro:thruster_macro thruster_id="4">
-    <origin xyz="0.3965 0.06271 -0.23105" rpy="${0*d2r} ${90.0*d2r} ${0*d2r}"/>
-  </xacro:thruster_macro>
-  <!-- Thruster 5 - Horizontal Back Left -->
-  <xacro:thruster_macro thruster_id="5">
-    <origin xyz="0.29505 0.06907 -0.16581" rpy="${0*d2r} ${90.0*d2r} ${0*d2r}"/>
-  </xacro:thruster_macro>
-  <!-- Thruster 6 - Vertical Front Left -->
-  <xacro:thruster_macro thruster_id="6">
-    <origin xyz="0.39685 0.06564 0.22015" rpy="${0*d2r} ${90.0*d2r} ${0*d2r}"/>
-  </xacro:thruster_macro>
-  <!-- Thruster 7 - Horizontal Front Left -->
-  <xacro:thruster_macro thruster_id="7">
-    <origin xyz="0.30146 0.06198 0.14961" rpy="${0*d2r} ${90.0*d2r} ${0*d2r}"/>
-  </xacro:thruster_macro>
  <!-- Default joint state publisher -->
  <gazebo>

Commit message: u-turn"

File: urdf/robots/lanturn_description/urdf/lanturn.xacro (robot description, xacro)
@@ -29,5 +29,5 @@
     </inertial>
     <visual>
-      <origin xyz="0 0 0" rpy="0 0 1.5708"/>
+      <origin xyz="0 0 0" rpy="0 0 0"/>
       <geometry>
         <mesh filename="package://lanturn_description/meshes/lanturn.dae" scale="1 1 1"/>
@@ -35,5 +35,5 @@
     </visual>
     <collision>
-      <origin xyz="0 0 0" rpy="0 0 1.5708"/>
+      <origin xyz="0 0 0" rpy="0 0 0"/>
       <geometry>
         <mesh filename="package://lanturn_description/meshes/lanturn.dae" scale="1 1 1"/>
@@ -128,19 +128,35 @@
   <!-- Forward:     Front   -->
   <!-- Aft:         Rear    -->
-  <!-- Thruster 0 - Vertical Starboard-Forward -->
-  <xacro:thruster_macro thruster_id="0">
-    <origin xyz="0.385 0.22 0.041" rpy="${0*d2r} ${-90*d2r} ${0*d2r}"/>
+  <!-- Thruster 1 - Vertical Port-Forward -->
+  <xacro:thruster_macro thruster_id="1">
+    <origin xyz="0.22 0.385 0.041" rpy="${0*d2r} ${-90*d2r} ${0*d2r}"/>
   </xacro:thruster_macro>
-  <!-- Thruster 1 - Vertical Starboard-Aft -->
-  <xacro:thruster_macro thruster_id="1">
-    <origin xyz="0.385 -0.22 0.041" rpy="${0*d2r} ${-90*d2r} ${0*d2r}"/>
-  </xacro:thruster_macro>
-  <!-- Thruster 2 - Vertical Port-Forward -->
+  <!-- Thruster 2 - Vertical Starboard-Forward -->
   <xacro:thruster_macro thruster_id="2">
-    <origin xyz="-0.385 0.22 0.041" rpy="${0*d2r} ${-90*d2r} ${0*d2r}"/>
+    <origin xyz="0.22 -0.385 0.041" rpy="${0*d2r} ${-90*d2r} ${0*d2r}"/>
   </xacro:thruster_macro>
   <!-- Thruster 3 - Vertical Port-Aft -->
   <xacro:thruster_macro thruster_id="3">
-    <origin xyz="-0.385 -0.22 0.041" rpy="${0*d2r} ${-90*d2r} ${0*d2r}"/>
+    <origin xyz="-0.22 0.385 0.041" rpy="${0*d2r} ${-90*d2r} ${0*d2r}"/>
+  </xacro:thruster_macro>
+  <!-- Thruster 4 - Vertical Starboard-Aft -->
+  <xacro:thruster_macro thruster_id="4">
+    <origin xyz="-0.22 -0.385 0.041" rpy="${0*d2r} ${-90*d2r} ${0*d2r}"/>
+  </xacro:thruster_macro>
+  <!-- Thruster 5 - Horizontal Port-Forward -->
+  <xacro:thruster_macro thruster_id="5">
+    <origin xyz="0.153 0.305 0.0425" rpy="${0*d2r} ${0*d2r} ${-45*d2r}"/>
+  </xacro:thruster_macro>
+  <!-- Thruster 6 - Horizontal Starboard-Forward -->
+  <xacro:thruster_macro thruster_id="6">
+    <origin xyz="0.153 -0.305 0.0425" rpy="${0*d2r} ${0*d2r} ${45*d2r}"/>
+  </xacro:thruster_macro>
+  <!-- Thruster 7 - Horizontal Port-Aft -->
+  <xacro:thruster_macro thruster_id="7">
+    <origin xyz="-0.153 0.305 0.0425" rpy="${0*d2r} ${0*d2r} ${45*d2r}"/>
+  </xacro:thruster_macro>
+  <!-- Thruster 8 - Horizontal Starboard-Aft -->
+  <xacro:thruster_macro thruster_id="8">
+    <origin xyz="-0.153 -0.305 0.0425" rpy="${0*d2r} ${0*d2r} ${-45*d2r}"/>
   </xacro:thruster_macro>
  <!-- Default joint state publisher -->
