Commit message: extra lanturn files

File: urdf/robots/lanturn_description/urdf/rexrov_oberon7.xacro (robot description, xacro)
@@ -17,6 +17,7 @@
   <xacro:arg name="inertial_reference_frame" default="world"/>
   <!-- Include the ROV macro file -->
-  <xacro:include filename="$(find lanturn_description)/urdf/lanturn_base.xacro"/>
+  <xacro:include filename="$(find rexrov_description)/urdf/rexrov_base.xacro"/>
   <xacro:include filename="$(find uuv_descriptions)/urdf/rexrov.gazebo.xacro"/>
+  <xacro:include filename="$(find dave_oberon7_description)/urdf/oberon7_default.xacro" />
   <!-- This implements the image_sonar_ros_plugin.so implemented in uuv_simulator.
        See the source code https://github.com/uuvsimulator/uuv_simulator/blob/master/uuv_sensor_plugins/uuv_sensor_ros_plugins/src/gazebo_ros_image_sonar.cpp
@@ -79,4 +80,7 @@
     </gazebo>
   </xacro:rexrov_base>
+  <xacro:oberon7 namespace="oberon7" parent="$(arg namespace)/base_link">
+    <origin xyz="1.3 -0.5 -0.615" rpy="0 0 0"/>
+  </xacro:oberon7>
   <gazebo>
       <plugin name="gazebo_ros_control" filename="libgazebo_ros_control.so">

File: urdf/robots/lanturn_description/urdf/rexrov_oberon7_sl3.xacro (robot description, xacro)
@@ -17,13 +17,8 @@
   <xacro:arg name="inertial_reference_frame" default="world"/>
   <!-- Include the ROV macro file -->
-  <xacro:include filename="$(find lanturn_description)/urdf/lanturn_base.xacro"/>
+  <xacro:include filename="$(find rexrov_description)/urdf/rexrov_base.xacro"/>
   <xacro:include filename="$(find uuv_descriptions)/urdf/rexrov.gazebo.xacro"/>
-  <!-- This implements the image_sonar_ros_plugin.so implemented in uuv_simulator.
-       See the source code https://github.com/uuvsimulator/uuv_simulator/blob/master/uuv_sensor_plugins/uuv_sensor_ros_plugins/src/gazebo_ros_image_sonar.cpp
-       See description wiki https://github.com/Field-Robotics-Lab/dave/wiki/image_sonar_description
-  -->
-  <!--  Commenting this out b/c the primary multibeam sonar sensor plugin is now here: https://github.com/Field-Robotics-Lab/nps_uw_multibeam_sonar
-       Keeping the snippet around for posterity -->
-  <!--
+  <xacro:include filename="$(find dave_oberon7_description)/urdf/oberon7_default.xacro" />
+  <xacro:include filename="$(find lidar_3dad_sl3_description)/urdf/sl3_lidar.xacro"/>
   <xacro:uuv_forward_looking_sonar
       namespace="${namespace}"
@@ -38,9 +33,9 @@
         height="492">
       <inertia ixx="0.00001" ixy="0.0" ixz="0.0" iyy="0.00001" iyz="0.0" izz="0.00001" />
+      <!--origin xyz="0.83 0 -0.22" rpy="0 ${0.2*pi} 0" /-->
       <origin xyz="1.15 0 0.4" rpy="0 0.3 0"/>
       <visual>
       </visual>
     </xacro:uuv_forward_looking_sonar>
-  -->
 <!--
   <xacro:uuv_forward_multibeam_p900
@@ -60,5 +55,5 @@
   <xacro:uuv_forward_multibeam_sonar_m450_130 namespace="$(arg namespace)" parent_link="$(arg namespace)/base_link">
     <origin xyz="1.4 0 0.65" rpy="0 0 0"/>
-  </xacro:uuv_forward_multibeam_sonar_m450_130>
+  </xacro:uuv_forward_multibeam_sonar_m450_130>e)
 -->
   <!-- Create the ROV -->
@@ -79,4 +74,12 @@
     </gazebo>
   </xacro:rexrov_base>
+  <xacro:oberon7 namespace="oberon7" parent="$(arg namespace)/base_link">
+    <origin xyz="1.3 -0.5 -0.615" rpy="0 0 0"/>
+  </xacro:oberon7>
+  <xacro:sl3_macro namespace="sl3" parent_link="$(arg namespace)/base_link"
+                   inertial_reference_frame="$(arg inertial_reference_frame)"
+                   pan="0" tilt="0">
+    <origin xyz="1.05 0 0.81" rpy="0 0 ${pi/2}"/>
+  </xacro:sl3_macro>
   <gazebo>
       <plugin name="gazebo_ros_control" filename="libgazebo_ros_control.so">

File: urdf/robots/lanturn_description/urdf/rexrov_oberon7_transient_current.xacro (robot description, xacro)
@@ -17,6 +17,7 @@
   <xacro:arg name="inertial_reference_frame" default="world"/>
   <!-- Include the ROV macro file -->
-  <xacro:include filename="$(find lanturn_description)/urdf/lanturn_base.xacro"/>
+  <xacro:include filename="$(find rexrov_description)/urdf/rexrov_base.xacro"/>
   <xacro:include filename="$(find uuv_descriptions)/urdf/rexrov.gazebo.xacro"/>
+  <xacro:include filename="$(find dave_oberon7_description)/urdf/oberon7_default.xacro" />
   <!-- This implements the image_sonar_ros_plugin.so implemented in uuv_simulator.
        See the source code https://github.com/uuvsimulator/uuv_simulator/blob/master/uuv_sensor_plugins/uuv_sensor_ros_plugins/src/gazebo_ros_image_sonar.cpp
@@ -69,7 +70,27 @@
      allow the addition of external models of manipulator units -->
     <gazebo>
+      <plugin name="dave_transient_current_plugin" filename="libdave_ocean_current_model_plugin.so">
+        <flow_velocity_topic>hydrodynamics/current_velocity/$(arg namespace)</flow_velocity_topic>
+        <base_link_name>$(arg namespace)/base_link</base_link_name>
+        <transient_current>
+          <topic_stratified>stratified_current_velocity</topic_stratified>
+          <velocity_north>
+            <noiseAmp>0.3</noiseAmp>
+            <noiseFreq>0.0</noiseFreq>
+          </velocity_north>
+          <velocity_east>
+            <noiseAmp>0.3</noiseAmp>
+            <noiseFreq>0.0</noiseFreq>
+          </velocity_east>
+          <velocity_down>
+            <noiseAmp>0.3</noiseAmp>
+            <noiseFreq>0.0</noiseFreq>
+          </velocity_down>
+        </transient_current>
+        <tide_oscillation>true</tide_oscillation>
+      </plugin>
       <plugin name="uuv_plugin" filename="libuuv_underwater_object_ros_plugin.so">
         <fluid_density>1028.0</fluid_density>
-        <flow_velocity_topic>hydrodynamics/current_velocity</flow_velocity_topic>
+        <flow_velocity_topic>hydrodynamics/current_velocity/$(arg namespace)</flow_velocity_topic>
         <debug>$(arg debug)</debug>
         <!-- Adding the hydrodynamic and hydrostatic parameters for the vehicle-->
@@ -79,4 +100,7 @@
     </gazebo>
   </xacro:rexrov_base>
+  <xacro:oberon7 namespace="oberon7" parent="$(arg namespace)/base_link">
+    <origin xyz="1.3 -0.5 -0.615" rpy="0 0 0"/>
+  </xacro:oberon7>
   <gazebo>
       <plugin name="gazebo_ros_control" filename="libgazebo_ros_control.so">

File: urdf/robots/lanturn_description/urdf/rexrov_predator.xacro (robot description, xacro)
@@ -17,13 +17,7 @@
   <xacro:arg name="inertial_reference_frame" default="world"/>
   <!-- Include the ROV macro file -->
-  <xacro:include filename="$(find lanturn_description)/urdf/lanturn_base.xacro"/>
+  <xacro:include filename="$(find rexrov_description)/urdf/rexrov_base.xacro"/>
   <xacro:include filename="$(find uuv_descriptions)/urdf/rexrov.gazebo.xacro"/>
-  <!-- This implements the image_sonar_ros_plugin.so implemented in uuv_simulator.
-       See the source code https://github.com/uuvsimulator/uuv_simulator/blob/master/uuv_sensor_plugins/uuv_sensor_ros_plugins/src/gazebo_ros_image_sonar.cpp
-       See description wiki https://github.com/Field-Robotics-Lab/dave/wiki/image_sonar_description
-  -->
-  <!--  Commenting this out b/c the primary multibeam sonar sensor plugin is now here: https://github.com/Field-Robotics-Lab/nps_uw_multibeam_sonar
-       Keeping the snippet around for posterity -->
-  <!--
+  <xacro:include filename="$(find predator_description)/urdf/predator_default.xacro" />
   <xacro:uuv_forward_looking_sonar
       namespace="${namespace}"
@@ -38,9 +32,9 @@
         height="492">
       <inertia ixx="0.00001" ixy="0.0" ixz="0.0" iyy="0.00001" iyz="0.0" izz="0.00001" />
+      <!--origin xyz="0.83 0 -0.22" rpy="0 ${0.2*pi} 0" /-->
       <origin xyz="1.15 0 0.4" rpy="0 0.3 0"/>
       <visual>
       </visual>
     </xacro:uuv_forward_looking_sonar>
-  -->
 <!--
   <xacro:uuv_forward_multibeam_p900
@@ -79,4 +73,7 @@
     </gazebo>
   </xacro:rexrov_base>
+  <xacro:predator namespace="predator" parent="$(arg namespace)/base_link">
+    <origin xyz="1.15 -0.5 -0.7" rpy="0 0 0"/>
+  </xacro:predator>
   <gazebo>
       <plugin name="gazebo_ros_control" filename="libgazebo_ros_control.so">
