Commit message: full lanturn description --pretest

File: lanturn/lanturn_description/urdf/lanturn_actuators.xacro (robot description, xacro)
@@ -8,4 +8,5 @@
           aware that Gazebo does not use the SNAME convention per default.
     -->
+    <!-- Temp comment out thrusters
     <xacro:thruster_macro robot_namespace="${namespace}" thruster_id="0">
         <origin xyz="0 0 0" rpy="0 0 ${pi}" />
@@ -17,16 +18,4 @@
     <origin xyz="0 0 0" rpy="0 -${0.5*pi} 0" />
     </xacro:thruster_macro>
-    <!-- Instantiate fins, if necessary -->
-    <xacro:fin_macro namespace="${namespace}" fin_id="0">
-      <origin xyz="0 0 0" rpy="0 0 0" />
-    </xacro:fin_macro>
-    <xacro:fin_macro namespace="${namespace}" fin_id="1">
-      <origin xyz="0 0 0" rpy="0 0 0" />
-    </xacro:fin_macro>
-    <xacro:fin_macro namespace="${namespace}" fin_id="2">
-      <origin xyz="0 0 0" rpy="0 0 0" />
-    </xacro:fin_macro>
-    <xacro:fin_macro namespace="${namespace}" fin_id="3">
-      <origin xyz="0 0 0" rpy="0 0 0" />
-    </xacro:fin_macro>
+    -->
 </robot>

File: lanturn/lanturn_description/urdf/lanturn_base.xacro (robot description, xacro)
@@ -23,9 +23,9 @@
     Open the meshes for the RexROV vehicle in Blender to see an example on the mesh placement.
   -->
-  <xacro:property name="visual_mesh_file" value="file://$(find lanturn_description)/meshes/vehicle.dae"/>
+  <xacro:property name="visual_mesh_file" value="file://$(find lanturn_description)/meshes/lanturn_no_prop.dae"/>
   <!-- Collision geometry mesh, usually in STL format (it is recommended to keep
   this geometry as simple as possible to improve the performance the physics engine
   regarding the computation of collision forces) -->
-  <xacro:property name="collision_mesh_file" value="file://$(find lanturn_description)/meshes/vehicle.stl"/>
+  <xacro:property name="collision_mesh_file" value="file://$(find lanturn_description)/meshes/lanturn_no_prop.dae"/>
   <!-- Vehicle macro -->
   <xacro:macro name="lanturn_base" params="namespace *gazebo">
@@ -62,7 +62,7 @@
     <xacro:insert_block name="gazebo"/>
     <!-- Include the thruster modules -->
-    <xacro:include filename="$(find lanturn_description)/urdf/actuators.xacro"/>
+    <xacro:include filename="$(find lanturn_description)/urdf/lanturn_actuators.xacro"/>
     <!-- Include the sensor modules -->
-    <xacro:include filename="$(find lanturn_description)/urdf/sensors.xacro"/>
+    <xacro:include filename="$(find lanturn_description)/urdf/lanturn_sensors.xacro"/>
   </xacro:macro>
 </robot>

File: lanturn/lanturn_description/urdf/lanturn_sensors.xacro (robot description, xacro)
@@ -7,8 +7,4 @@
     more examples or add you own custom sensor units.
   -->
-  <!-- Mount a GPS. -->
-  <xacro:default_gps namespace="${namespace}" parent_link="${namespace}/base_link" />
-  <!-- Mount a Pose 3D sensor. -->
-  <xacro:default_pose_3d namespace="${namespace}" parent_link="${namespace}/base_link" />
   <!-- Forward-looking sonar sensor -->
   <xacro:forward_multibeam_p900 namespace="${namespace}" parent_link="${namespace}/base_link">
@@ -19,8 +15,4 @@
     <origin xyz="0 0 0" rpy="0 0 0"/>
   </xacro:default_dvl>
-  <!-- RPT  -->
-  <xacro:default_rpt namespace="${namespace}" parent_link="${namespace}/base_link">
-    <origin xyz="0 0 0" rpy="0 0 0"/>
-  </xacro:default_rpt>
   <!-- Pressure  -->
   <xacro:default_pressure namespace="${namespace}" parent_link="${namespace}/base_link">
